File: PCB/Backplane/Backplane.kicad_pcb (KiCad board)
At the start: 2 copper layers, 551.8 x 66.4 mm, 29 parts

Commit message: update backplane PCB
Parts:
- removed the 0 at (493.5, 207.3)
- removed the 0 at (282.0, 207.3)
- removed the 0 at (211.5, 207.3)
- removed the 0 at (141.0, 207.3)
- removed the 0 at (423.0, 207.3)
- removed the 0 at (0.00, 207.3)
- removed the 0 at (70.5, 207.3)
- removed the 0 at (352.5, 207.3)
- removed the REF** at (151.0, 226.9)
- removed the REF** at (221.5, 226.9)
- removed the REF** at (151.0, 188.0)
- removed the REF** at (292.0, 226.9)
- removed the REF** at (80.5, 188.0)
- removed the REF** at (433.0, 188.0)
- removed the REF** at (362.5, 226.9)
- removed the REF** at (80.5, 226.9)
- removed the REF** at (503.5, 226.9)
- removed the REF** at (541.7, 192.6)
- removed the REF** at (503.5, 188.0)
- removed the REF** at (221.5, 188.0)
- removed the REF** at (292.0, 188.0)
- removed the REF** at (433.0, 226.9)
- removed the REF** at (362.5, 188.0)
- added 0: CONN12_2x06_DRXH_SUL, Custom Library:CONN12_2x06_DRXH_SUL, F.Cu at (449.7, 207.6)
- added 0: CONN12_2x06_DRXH_SUL, Custom Library:CONN12_2x06_DRXH_SUL, F.Cu at (520.2, 207.6)
- added 0: CONN12_2x06_DRXH_SUL, Custom Library:CONN12_2x06_DRXH_SUL, F.Cu at (379.2, 207.6)
- added 0: CONN12_2x06_DRXH_SUL, Custom Library:CONN12_2x06_DRXH_SUL, F.Cu at (97.2, 207.6)
- added 0: CONN12_2x06_DRXH_SUL, Custom Library:CONN12_2x06_DRXH_SUL, F.Cu at (26.7, 207.6)
- added 0: CONN12_2x06_DRXH_SUL, Custom Library:CONN12_2x06_DRXH_SUL, F.Cu at (167.7, 207.6)
- added 0: CONN12_2x06_DRXH_SUL, Custom Library:CONN12_2x06_DRXH_SUL, F.Cu at (238.2, 207.6)
- added 0: CONN12_2x06_DRXH_SUL, Custom Library:CONN12_2x06_DRXH_SUL, F.Cu at (308.7, 207.6)
- added A135914-ND: CONN2_282836-1_TEC, Custom Library:CONN2_282836-1_TEC, F.Cu at (567.6, 235.5)
- added JST XH 3: JST_XH_B3B-XH-A_1x03_P2.50mm_Vertical, Connector_JST:JST_XH_B3B-XH-A_1x03_P2.50mm_Vertical, F.Cu at (276.9, 241.3)
- added JST XH 3: JST_XH_B3B-XH-A_1x03_P2.50mm_Vertical, Connector_JST:JST_XH_B3B-XH-A_1x03_P2.50mm_Vertical, F.Cu at (297.2, 180.6)
- added REF**: MountingHole_3.2mm_M3, MountingHole:MountingHole_3.2mm_M3, F.Cu at (244.9, 228.9)
- added REF**: MountingHole_3.2mm_M3, MountingHole:MountingHole_3.2mm_M3, F.Cu at (385.9, 228.9)
- added REF**: MountingHole_3.2mm_M3, MountingHole:MountingHole_3.2mm_M3, F.Cu at (526.9, 199.0)
- added REF**: MountingHole_3.2mm_M3, MountingHole:MountingHole_3.2mm_M3, F.Cu at (315.4, 199.0)
- added REF**: MountingHole_3.2mm_M3, MountingHole:MountingHole_3.2mm_M3, F.Cu at (103.9, 199.0)
- added REF**: MountingHole_3.2mm_M3, MountingHole:MountingHole_3.2mm_M3, F.Cu at (103.9, 228.9)
- added REF**: MountingHole_3.2mm_M3, MountingHole:MountingHole_3.2mm_M3, F.Cu at (385.9, 199.0)
- added REF**: MountingHole_3.2mm_M3, MountingHole:MountingHole_3.2mm_M3, F.Cu at (526.9, 228.9)
- added REF**: MountingHole_3.2mm_M3, MountingHole:MountingHole_3.2mm_M3, F.Cu at (174.4, 228.9)
- added REF**: MountingHole_3.2mm_M3, MountingHole:MountingHole_3.2mm_M3, F.Cu at (456.4, 228.9)
- added REF**: MountingHole_3.2mm_M3, MountingHole:MountingHole_3.2mm_M3, F.Cu at (174.4, 199.0)
- added REF**: MountingHole_3.2mm_M3, MountingHole:MountingHole_3.2mm_M3, F.Cu at (456.4, 199.0)
- added REF**: MountingHole_3.2mm_M3, MountingHole:MountingHole_3.2mm_M3, F.Cu at (244.9, 199.0)
- added REF**: MountingHole_3.2mm_M3, MountingHole:MountingHole_3.2mm_M3, F.Cu at (315.4, 228.9)
- REF** (x2): value PinHeader_2x17_P2.54mm_Vertical -> PinSocket_2x17_P2.54mm_Vertical; footprint Connector_PinHeader_2.54mm:PinHeader_2x17_P2.54mm_Vertical -> Connector_PinSocket_2.54mm:PinSocket_2x17_P2.54mm_Vertical
- moved 100µF 37.2 mm to (553.7, 228.2)
- moved REF** 25.9 mm to (33.4, 199.0)
- moved REF** 25.2 mm to (280.7, 221.9)
- moved REF** 25.2 mm to (262.9, 221.9)
- moved REF** 23.5 mm to (33.4, 228.9)
- moved R-78K5.0 9.82 mm to (533.5, 213.0)
- renumbered REF** to R-78K5.0
Connections:
- REF** pad 17: (no net) -> Step_5
- REF** pad 18: (no net) -> Step_5
- REF** pad 19: (no net) -> Step_4
- REF** pad 20: (no net) -> Step_4
- REF** pad 5: Step_5 -> (no net)
- REF** pad 6: Step_5 -> (no net)
- REF** pad 7: Step_4 -> (no net)
- REF** pad 8: Step_4 -> (no net)
Routing:
- net +12V: track 564.4 -> 823.0 mm
- net SDA: track 2.54 -> 74.3 mm
- net SCL: track 2.54 -> 74.3 mm
- net GND: track 45.8 -> 81.3 mm, vias 16 -> 24
- net +5V: track 563.9 -> 549.5 mm
- net Step_5: track 129.5 -> 137.8 mm
- net Step_4: track 30.5 -> 34.7 mm
- net Hall_3: track 28.2 -> 31.9 mm
- net Step_6: track 198.9 -> 195.4 mm
- net Step_7: track 268.7 -> 265.2 mm
- net Hall_2: track 107.9 -> 104.5 mm
- net Hall_1: track 178.4 -> 176.0 mm
- net Step_0: track 262.4 -> 264.6 mm
- net Step_1: track 192.7 -> 194.8 mm
- net Step_2: track 137.8 -> 140.0 mm
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Other:
- board size 551.8 x 66.4 mm -> 555.6 x 66.4 mm
- board text added: "BLK"
- board text added: "EBC06DRXH"
- board text added: "ORA"
- board text added: "SCL"
- board text added: "SDA"
- board text added: "Split Flap Back Plane V4 Stefan Frech"
- board text added: "YLW"
- board text removed: "Split Flap Back Plane V3 Stefan Frech"

Commit message: update backplane PCB with I2C connectors and new 3D models
Parts:
- removed A135914-ND: CONN2_282836-1_TEC, Custom Library:CONN2_282836-1_TEC
- removed R-78K5.0: Converter_DCDC_RECOM_R-78E-0.5_THT, Converter_DCDC:Converter_DCDC_RECOM_R-78E-0.5_THT
- added REF**: CONN2_282836-1_TEC, Library:CONN2_282836-1_TEC, F.Cu at (567.6, 235.5)
- added REF**: CONV_R-78K5.0-1.0, Converter_DCDC:CONV_R-78K5.0-1.0, F.Cu at (535.9, 214.6)
- moved JST XH 3 21.7 mm to (275.6, 179.1), turned to 180 degrees
- moved JST XH 3 6.44 mm to (270.6, 240.0), turned to 0 degrees
- moved REF** 6.32 mm to (262.9, 228.2)
- moved REF** 6.32 mm to (280.7, 228.2)
Connections:
- JST XH 3 pad 1: SDA -> GND
- JST XH 3 pad 3: GND -> SDA
Routing:
- net Step_2: track 140.0 -> 128.9 mm
- net Step_1: track 194.8 -> 185.5 mm
- net Step_6: track 195.4 -> 186.3 mm
- net Step_0: track 264.6 -> 255.8 mm
- net Step_7: track 265.2 -> 256.8 mm
- net +5V: track 549.5 -> 557.3 mm
- net Step_5: track 137.8 -> 130.6 mm
- net SDA: track 74.3 -> 69.8 mm
- net SCL: track 74.3 -> 69.8 mm
- net Hall_3: track 31.9 -> 29.2 mm
- net Step_3: track 34.0 -> 31.3 mm
- net Hall_7: track 250.4 -> 247.9 mm
- net Step_4: track 34.7 -> 32.1 mm
- net Hall_6: track 178.9 -> 176.3 mm
- net Hall_5: track 107.3 -> 104.8 mm
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Other:
- board size 555.6 x 66.4 mm -> 555.6 x 69 mm
- board text added: "282836-1"
- board text added: "BLK GND"
- board text added: "ORA SCL"
- board text added: "Split Flap Back Plane V5 Stefan Frech"
- board text added: "YLW SDA"
- board text removed: "BLK"
- board text removed: "ORA"
- board text removed: "SCL"
- board text removed: "SDA"
- board text removed: "Split Flap Back Plane V4 Stefan Frech"
- board text removed: "YLW"
